File: Hardware/Qwiic AHT20 Breakout.brd (EAGLE design)
At the start: 25.4 x 25.4 mm, 38 parts, among them J2 QWIIC_RIGHT_ANGLE, J3 PTH, J4 QWIIC_RIGHT_ANGLE, U2 AHT20QFN-6

Commit message: Added NCD2400M to schematic
Parts:
- removed U2: AHT20QFN-6, AHT20:QFN-6
- added U1: NCD2400MDFN, SparkFun-Capacitors:DFN6
Connections:
- net 3.3V: now also U1.4; no longer U2.VDD
- net GND: now also U1.5; no longer U2.GND
- net SCL: now also U1.1; no longer U2.SCL
- net SDA: now also U1.6; no longer U2.SDA
Routing:
- net GND: track 5.99 -> 0.14 mm, vias 5 -> 4
- net SDA: track 42.2 -> 38.0 mm
- net SCL: track 49.3 -> 47.1 mm
Changed lines of the file:
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@@
 <?xml version="1.0" encoding="utf-8"?>
 <!DOCTYPE eagle SYSTEM "eagle.dtd">
-<eagle version="9.6.0">
+<eagle version="9.5.2">
 <drawing>
 <settings>
-<setting alwaysvectorfont="yes"/>
+<setting alwaysvectorfont="no"/>
 <setting keepoldvectorfont="yes"/>
 <setting verticaltext="up"/>
@@
 <attribute name="VALUE" x="6.35" y="9.398" size="0.6096" layer="28" font="vector" ratio="20" rot="MR180" align="top-center"/>
 </element>
-<element name="U2" library="AHT20" package="QFN-6" value="AHT20QFN-6" x="12.7" y="12.7" smashed="yes">
-<attribute name="NAME" x="12.7" y="14.605" size="0.6096" layer="25" font="vector" ratio="20" align="bottom-center"/>
-<attribute name="PROD_ID" value="IC-" x="12.7" y="12.7" size="1.778" layer="27" font="vector" ratio="15" display="off"/>
-<attribute name="VALUE" x="12.7" y="11.049" size="0.6096" layer="27" font="vector" ratio="20" align="top-center"/>
-</element>
 <element name="U$14" library="buzzard_labels (17)" package="AHT20_HUMIDITY2" value="" x="5.969" y="21.209" smashed="yes"/>
 <element name="U$12" library="SparkFun-Buzzard" package="LED_32" value="" x="8.128" y="6.223" smashed="yes" rot="MR0"/>
 <element name="U$18" library="SparkFun-Aesthetics" package="ORDERING_INSTRUCTIONS" value="" x="39.37" y="50.8" smashed="yes"/>
 <element name="U$8" library="buzzard_labels (17)" package="AHT20_HUMIDITY2" value="" x="19.304" y="21.209" smashed="yes" rot="MR0"/>
+<element name="U1" library="SparkFun-Capacitors" package="DFN6" value="NCD2400MDFN" x="-31.75" y="-21.59" smashed="yes">
+<attribute name="NAME" x="-32.385" y="-21.082" size="0.254" layer="25"/>
+<attribute name="VALUE" x="-32.385" y="-22.352" size="0.254" layer="27"/>
+</element>
 </elements>
 <signals>
@@
 <contactref element="C1" pad="1"/>
 <contactref element="LED" pad="2"/>
-<contactref element="U2" pad="VDD"/>
-<wire x1="11.7" y1="12.7" x2="11.811" y2="12.7" width="0.1524" layer="1"/>
 <wire x1="11.85" y1="9.13294375" x2="11.85" y2="7.62" width="0.1524" layer="1"/>
 <wire x1="5.08" y1="13.2" x2="6.977" y2="13.2" width="0.3048" layer="1"/>
@@
 <wire x1="12.446" y1="12.065" x2="12.446" y2="9.72894375" width="0.1524" layer="1"/>
 <wire x1="12.446" y1="9.72894375" x2="11.85" y2="9.13294375" width="0.1524" layer="1"/>
+<contactref element="U1" pad="4"/>
+<wire x1="11.43" y1="1.27" x2="-30.6959" y2="-22.2504" width="0" layer="19" extent="1-1"/>
 </signal>
 <signal name="GND">
@@
 <contactref element="J2" pad="1"/>
 <contactref element="J4" pad="1"/>
-<contactref element="U2" pad="GND"/>
-<wire x1="13.7" y1="12.7" x2="13.319" y2="12.7" width="0.1524" layer="1"/>
-<wire x1="13.319" y1="12.7" x2="12.7254" y2="13.2936" width="0.1524" layer="1"/>
-<wire x1="12.7254" y1="13.2936" x2="12.7254" y2="13.716" width="0.1524" layer="1"/>
-<via x="12.7254" y="13.716" extent="1-16" drill="0.3048"/>
 <via x="14.605" y="7.493" extent="1-16" drill="0.3048"/>
 <via x="19.05" y="11.176" extent="1-16" drill="0.3048"/>
@@
 <via x="3.683" y="14.224" extent="1-16" drill="0.3048"/>
 <wire x1="13.2334" y1="9.6266" x2="13.335" y2="9.525" width="0.1524" layer="16"/>
-<wire x1="12.7254" y1="13.716" x2="12.7" y2="13.6906" width="0.1524" layer="16"/>
-<wire x1="12.7" y1="13.6906" x2="12.7" y2="9.525" width="0.1524" layer="16"/>
+<contactref element="U1" pad="5"/>
+<wire x1="3.417" y1="6.985" x2="-30.6959" y2="-21.59" width="0" layer="19" extent="1-1"/>
+<wire x1="4.699" y1="6.985" x2="3.417" y2="6.985" width="0" layer="19" extent="1-1"/>
+<wire x1="8.89" y1="1.27" x2="4.699" y2="6.985" width="0" layer="19" extent="1-1"/>
+<wire x1="5.08" y1="14.2" x2="4.699" y2="6.985" width="0" layer="19" extent="1-1"/>
+<wire x1="3.683" y1="14.224" x2="5.08" y2="14.2" width="0" layer="19" extent="1-1"/>
+<wire x1="13.55" y1="7.62" x2="8.89" y2="1.27" width="0" layer="19" extent="1-1"/>
+<wire x1="14.605" y1="7.493" x2="13.55" y2="7.62" width="0" layer="19" extent="1-1"/>
+<wire x1="13.335" y1="9.525" x2="13.55" y2="7.62" width="0" layer="19" extent="1-16"/>
+<wire x1="19.05" y1="11.176" x2="14.605" y2="7.493" width="0" layer="19" extent="1-1"/>
+<wire x1="20.32" y1="11.2" x2="19.05" y2="11.176" width="0" layer="19" extent="1-1"/>
 </signal>
 <signal name="SCL">
@@
 <contactref element="J3" pad="4"/>
 <contactref element="J4" pad="4"/>
-<contactref element="R1" pad="1"/>
-<contactref element="U2" pad="SCL"/>
-<wire x1="11.7" y1="11.7" x2="11.8204" y2="11.7" width="0.1524" layer="1"/>
 <wire x1="11.8204" y1="11.7" x2="12.1412" y2="11.3792" width="0.1524" layer="1"/>
 <wire x1="5.08" y1="11.2" x2="6.9102" y2="11.2" width="0.1524" layer="1"/>
@@
 <wire x1="12.1412" y1="9.8552" x2="11.303" y2="9.017" width="0.1524" layer="1"/>
 <wire x1="12.1412" y1="11.3792" x2="12.1412" y2="9.8552" width="0.1524" layer="1"/>
-<wire x1="9.74" y1="16.51" x2="11.811" y2="16.51" width="0.1524" layer="1"/>
 <wire x1="11.811" y1="16.51" x2="13.843" y2="18.542" width="0.1524" layer="1"/>
 <wire x1="13.843" y1="18.542" x2="16.256" y2="18.542" width="0.1524" layer="1"/>
 <wire x1="16.256" y1="18.542" x2="16.51" y2="18.288" width="0.1524" layer="1"/>
 <wire x1="16.51" y1="18.288" x2="16.51" y2="15.367" width="0.1524" layer="1"/>
+<contactref element="U1" pad="1"/>
+<contactref element="R1" pad="1"/>
+<wire x1="5.08" y1="11.2" x2="-32.8041" y2="-20.9296" width="0" layer="19" extent="1-1"/>
+<wire x1="9.74" y1="16.51" x2="11.811" y2="16.51" width="0" layer="19" extent="1-1"/>
 </signal>
 <signal name="SDA">
@@
 <contactref element="J3" pad="3"/>
 <contactref element="J4" pad="3"/>
-<contactref element="R2" pad="1"/>
-<contactref element="U2" pad="SDA"/>
 <wire x1="5.08" y1="12.2" x2="7.612" y2="12.2" width="0.1524" layer="1"/>
 <wire x1="7.612" y1="12.2" x2="8.89" y2="10.922" width="0.1524" layer="1"/>
@@
 <wire x1="15.24" y1="8.89" x2="16.51" y2="8.89" width="0.1524" layer="1"/>
 <wire x1="16.51" y1="8.89" x2="17.78" y2="10.16" width="0.1524" layer="1"/>
-<wire x1="17.36" y1="16.51" x2="21.463" y2="16.51" width="0.1524" layer="1"/>
 <wire x1="21.463" y1="16.51" x2="22.225" y2="15.748" width="0.1524" layer="1"/>
 <wire x1="22.225" y1="15.748" x2="22.225" y2="13.97" width="0.1524" layer="1"/>
@@
 <wire x1="8.89" y1="8.89" x2="8.89" y2="8.83994375" width="0.1524" layer="16"/>
 <wire x1="9.50034375" y1="8.2296" x2="12.92094375" y2="8.2296" width="0.1524" layer="16"/>
-<wire x1="13.7" y1="11.7" x2="13.5288" y2="11.7" width="0.1524" layer="1"/>
 <wire x1="13.5288" y1="11.7" x2="13.2588" y2="11.43" width="0.1524" layer="1"/>
 <wire x1="13.2588" y1="11.43" x2="13.2588" y2="10.16" width="0.1524" layer="1"/>
@@
 <wire x1="13.2588" y1="9.65274375" x2="13.2588" y2="9.6012" width="0.1524" layer="1"/>
 <wire x1="13.2588" y1="9.6012" x2="13.97" y2="8.89" width="0.1524" layer="1"/>
+<contactref element="U1" pad="6"/>
+<contactref element="R2" pad="1"/>
+<wire x1="5.08" y1="12.2" x2="-30.6959" y2="-20.9296" width="0" layer="19" extent="1-1"/>
+<wire x1="17.36" y1="16.51" x2="21.463" y2="16.51" width="0" layer="19" extent="1-1"/>
 </signal>
 <signal name="N$3">
