File: Hardware/Qwiic_I2C_Capacitor.sch (EAGLE design)
At the start: 23 parts, among them J2 QWIIC_RIGHT_ANGLE, J3 PTH, J4 QWIIC_RIGHT_ANGLE, U1 NCD2400MDFN

Commit message: Renamed eagle files
Other:
- note added: "Priyanka Makin"
Changed lines of the file:
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@@
 <wire x1="0" y1="68.58" x2="248.92" y2="68.58" width="0.2032" layer="97" style="longdash"/>
 <text x="63.5" y="60.96" size="2.54" layer="97" align="center">Connectors</text>
+<text x="167.64" y="10.16" size="2.54" layer="94">Priyanka Makin</text>
 </plain>
 <instances>

Commit message: Update Qwiic_I2C_Capacitor.sch
Other:
- note added: "I2C Address for NCD2400M: 0x60 I2C Address for NCD2400M1: 0x61"
Changed lines of the file:
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@@
 <?xml version="1.0" encoding="utf-8"?>
 <!DOCTYPE eagle SYSTEM "eagle.dtd">
-<eagle version="9.5.2">
+<eagle version="9.4.2">
 <drawing>
 <settings>
-<setting alwaysvectorfont="no"/>
+<setting alwaysvectorfont="yes"/>
 <setting keepoldvectorfont="yes"/>
 <setting verticaltext="up"/>
@@
 <text x="63.5" y="60.96" size="2.54" layer="97" align="center">Connectors</text>
 <text x="167.64" y="10.16" size="2.54" layer="94">Priyanka Makin</text>
+<text x="119.38" y="99.06" size="1.778" layer="97">I2C Address for NCD2400M: 0x60
+I2C Address for NCD2400M1: 0x61</text>
 </plain>
 <instances>
@@
 </drawing>
 <compatibility>
+<note version="6.3" minversion="6.2.2" severity="warning">
+Since Version 6.2.2 text objects can contain more than one line,
+which will not be processed correctly with this version.
+</note>
 <note version="8.3" severity="warning">
 Since Version 8.3, EAGLE supports URNs for individual library

Commit message: Initial layout
Parts:
- removed C1: 0.1uF, SparkFun-Capacitors:0.1UF-0603-25V-(+80/-20%)
- removed J4: QWIIC_RIGHT_ANGLE, SparkFun-Connectors:QWIIC_CONNECTORJS-1MM
- removed JP3, JP4, JP8, JP9: STAND-OFF, SparkFun-Hardware:STAND-OFF
- removed U$1, U$2: SPARKX-LOGO4, SparkX:SPARKX-LOGO4
- added J1: CONN_02_0603, Qwiic_Capacitor:CONN_02_0603
- JP1, JP2, JP5, JP6: value FIDUCIAL1X2 -> FIDUCIAL0.2MM; device SparkFun-Aesthetics:FIDUCIAL1X2 -> SparkFun-Aesthetics:FIDUCIAL0.2MM
Connections:
- new net CN: J1.2, U1.CN
- new net CP: J1.1, U1.CP
- net 3.3V: no longer C1.1, J4.2
- net GND: no longer C1.2, J4.1
- net SCL: no longer J4.4
- net SDA: no longer J4.3
Other:
- moved on the sheet: J2, J3

Commit message: Changes from board review
Parts:
- added LOGO2: SPECIAL_INSTRUCTIONS-ORDERING, SparkFun-Aesthetics:SPECIAL_INSTRUCTIONS-ORDERING
- added R4: 1k, SparkFun-Resistors:1KOHM-0603-1/10W-1%
- added R5: 10k, SparkFun-Resistors:10KOHM-0402T-1/16W-1%
Other:
- note added: "Digital Capacitor"
- note added: "Power LED"
- moved on the sheet: D1, J1, JP7, LED, R1, R2, R3, U1

Commit message: Panelizer/cam output
Parts:
- removed R4: 1k, SparkFun-Resistors:1KOHM-0603-1/10W-1%
- removed R5: 10k, SparkFun-Resistors:10KOHM-0402T-1/16W-1%
Changed lines of the file:
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@@
 <part name="LED" library="SparkFun-Jumpers" deviceset="JUMPER-SMT_2_NC_TRACE" device="_SILK" package3d_urn="urn:adsk.eagle:package:39281/1" value="JUMPER-SMT_2_NC_TRACE_SILK"/>
 <part name="U1" library="SparkFun-Capacitors" deviceset="NCD2400M" device="DFN"/>
-<part name="R4" library="SparkFun-Resistors" deviceset="1KOHM" device="-0603-1/10W-1%" value="1k"/>
-<part name="R5" library="SparkFun-Resistors" deviceset="10KOHM" device="-0402T-1/16W-1%" value="10k"/>
 <part name="LOGO2" library="SparkFun-Aesthetics" deviceset="SPECIAL_INSTRUCTIONS" device="-ORDERING"/>
 <part name="J1" library="Qwiic_Capacitor" deviceset="CONN_02_0603" device=""/>
@@
 <attribute name="VALUE" x="144.78" y="114.3" size="1.778" layer="95"/>
 </instance>
-<instance part="R4" gate="G$1" x="55.88" y="127" smashed="yes" rot="R90">
-<attribute name="NAME" x="54.356" y="127" size="1.778" layer="95" font="vector" rot="R90" align="bottom-center"/>
-<attribute name="VALUE" x="57.404" y="127" size="1.778" layer="96" font="vector" rot="R90" align="top-center"/>
-</instance>
-<instance part="R5" gate="G$1" x="60.96" y="93.98" smashed="yes">
-<attribute name="NAME" x="60.96" y="95.504" size="1.778" layer="95" font="vector" align="bottom-center"/>
-<attribute name="VALUE" x="60.96" y="92.456" size="1.778" layer="96" font="vector" align="top-center"/>
-</instance>
 <instance part="LOGO2" gate="G$1" x="226.06" y="33.02" smashed="yes"/>

Commit message: Rev x02
Re-routed SDA and SCL. They were backwards in the previous version x01
Connections:
- net SCL: now also R2.1, U1.SCL; no longer R1.1, U1.SDA
- net SDA: now also R1.1, U1.SDA; no longer R2.1, U1.SCL
Other:
- note added: "x02"
- note removed: "x01"
Changed lines of the file:
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@@
 <sheet>
 <plain>
-<text x="237.744" y="7.366" size="2.54" layer="94">x01</text>
+<text x="237.744" y="7.366" size="2.54" layer="94">x02</text>
 <text x="43.688" y="98.806" size="1.778" layer="97">Power</text>
 <wire x1="0" y1="68.58" x2="76.2" y2="68.58" width="0.2032" layer="97" style="longdash"/>
@@
 </segment>
 <segment>
-<wire x1="142.24" y1="124.46" x2="116.84" y2="124.46" width="0.1524" layer="91"/>
-<label x="111.76" y="124.46" size="1.27" layer="95" rot="R180" xref="yes"/>
-<pinref part="U1" gate="U1" pin="SDA"/>
-<pinref part="R1" gate="G$1" pin="1"/>
-<wire x1="116.84" y1="124.46" x2="111.76" y2="124.46" width="0.1524" layer="91"/>
-<wire x1="116.84" y1="129.54" x2="116.84" y2="124.46" width="0.1524" layer="91"/>
-<junction x="116.84" y="124.46"/>
+<pinref part="U1" gate="U1" pin="SCL"/>
+<wire x1="142.24" y1="119.38" x2="132.08" y2="119.38" width="0.1524" layer="91"/>
+<pinref part="R2" gate="G$1" pin="1"/>
+<wire x1="132.08" y1="119.38" x2="132.08" y2="129.54" width="0.1524" layer="91"/>
+<wire x1="132.08" y1="119.38" x2="114.3" y2="119.38" width="0.1524" layer="91"/>
+<junction x="132.08" y="119.38"/>
+<label x="114.3" y="119.38" size="1.27" layer="95" rot="R180" xref="yes"/>
 </segment>
 </net>
@@
 </segment>
 <segment>
-<wire x1="111.76" y1="119.38" x2="132.08" y2="119.38" width="0.1524" layer="91"/>
-<label x="111.76" y="119.38" size="1.27" layer="95" rot="R180" xref="yes"/>
-<pinref part="U1" gate="U1" pin="SCL"/>
-<pinref part="R2" gate="G$1" pin="1"/>
-<wire x1="132.08" y1="119.38" x2="142.24" y2="119.38" width="0.1524" layer="91"/>
-<wire x1="132.08" y1="129.54" x2="132.08" y2="119.38" width="0.1524" layer="91"/>
-<junction x="132.08" y="119.38"/>
+<pinref part="U1" gate="U1" pin="SDA"/>
+<wire x1="142.24" y1="124.46" x2="116.84" y2="124.46" width="0.1524" layer="91"/>
+<pinref part="R1" gate="G$1" pin="1"/>
+<wire x1="116.84" y1="124.46" x2="116.84" y2="129.54" width="0.1524" layer="91"/>
+<wire x1="116.84" y1="124.46" x2="114.3" y2="124.46" width="0.1524" layer="91"/>
+<junction x="116.84" y="124.46"/>
+<label x="114.3" y="124.46" size="1.27" layer="95" rot="R180" xref="yes"/>
 </segment>
 </net>
