File: Hardware/Production/Qwiic_I2C_Capacitor-Panel.brd (EAGLE design)
At the start: 85.9 x 84.6 mm, 821 parts, among them J1 CONN_02_0603, J10 QWIIC_RIGHT_ANGLE, J11 PTH, J12 CONN_02_0603, J13 QWIIC_RIGHT_ANGLE, J14 PTH, J15 CONN_02_0603, J16 QWIIC_RIGHT_ANGLE, J17 PTH, J18 CONN_02_0603, J19 QWIIC_RIGHT_ANGLE, J2 QWIIC_RIGHT_ANGLE, J20 PTH, J21 CONN_02_0603, J22 QWIIC_RIGHT_ANGLE, J23 PTH, J24 CONN_02_0603, J25 QWIIC_RIGHT_ANGLE, J26 PTH, J27 CONN_02_0603, J28 QWIIC_RIGHT_ANGLE, J29 PTH, J3 PTH, J30 CONN_02_0603, J31 QWIIC_RIGHT_ANGLE, J32 PTH, J33 CONN_02_0603, J34 QWIIC_RIGHT_ANGLE, J35 PTH, J36 CONN_02_0603, J37 QWIIC_RIGHT_ANGLE, J38 PTH, J39 CONN_02_0603, J4 QWIIC_RIGHT_ANGLE, J40 QWIIC_RIGHT_ANGLE, J41 PTH, J42 CONN_02_0603, J43 QWIIC_RIGHT_ANGLE, J44 PTH, J45 CONN_02_0603, J46 QWIIC_RIGHT_ANGLE, J47 PTH, J48 CONN_02_0603, J49 QWIIC_RIGHT_ANGLE, J5 PTH, J50 PTH, J51 CONN_02_0603, J52 QWIIC_RIGHT_ANGLE, J53 PTH, J54 CONN_02_0603, J55 QWIIC_RIGHT_ANGLE, J56 PTH, J57 CONN_02_0603, J58 QWIIC_RIGHT_ANGLE, J59 PTH, J6 CONN_02_0603, J60 CONN_02_0603, J61 QWIIC_RIGHT_ANGLE, J62 PTH, J63 CONN_02_0603, J64 QWIIC_RIGHT_ANGLE, J65 PTH, J66 CONN_02_0603, J67 QWIIC_RIGHT_ANGLE, J68 PTH, J69 CONN_02_0603, J7 QWIIC_RIGHT_ANGLE, J70 QWIIC_RIGHT_ANGLE, J71 PTH, J72 CONN_02_0603, J8 PTH, J9 CONN_02_0603, U1 NCD2400MDFN, U10 NCD2400MDFN, U11 NCD2400MDFN, U12 NCD2400MDFN, U13 NCD2400MDFN, U14 NCD2400MDFN, U15 NCD2400MDFN, U16 NCD2400MDFN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

Commit message: Rev x02
Re-routed SDA and SCL. They were backwards in the previous version x01
Parts:
- added E$6: (no value), SparkFun-Retired:FIDUCIAL-1.5X3
Connections:
- net SCL: now also R2.1, U1.6; no longer R1.1, U1.1
- net SCL1: now also R6.1, U2.6; no longer R5.1, U2.1
- net SCL10: now also R33.1, U11.6; no longer R32.1, U11.1
- net SCL11: now also R36.1, U12.6; no longer R35.1, U12.1
- net SCL12: now also R39.1, U13.6; no longer R38.1, U13.1
- net SCL13: now also R42.1, U14.6; no longer R41.1, U14.1
- net SCL14: now also R45.1, U15.6; no longer R44.1, U15.1
- net SCL15: now also R48.1, U16.6; no longer R47.1, U16.1
- net SCL16: now also R51.1, U17.6; no longer R50.1, U17.1
- net SCL17: now also R54.1, U18.6; no longer R53.1, U18.1
- net SCL18: now also R57.1, U19.6; no longer R56.1, U19.1
- net SCL19: now also R60.1, U20.6; no longer R59.1, U20.1
- net SCL2: now also R9.1, U3.6; no longer R8.1, U3.1
- net SCL20: now also R63.1, U21.6; no longer R62.1, U21.1
- net SCL21: now also R66.1, U22.6; no longer R65.1, U22.1
- net SCL22: now also R69.1, U23.6; no longer R68.1, U23.1
- net SCL23: now also R72.1, U24.6; no longer R71.1, U24.1
- net SCL3: now also R12.1, U4.6; no longer R11.1, U4.1
- net SCL4: now also R15.1, U5.6; no longer R14.1, U5.1
- net SCL5: now also R18.1, U6.6; no longer R17.1, U6.1
- net SCL6: now also R21.1, U7.6; no longer R20.1, U7.1
- net SCL7: now also R24.1, U8.6; no longer R23.1, U8.1
- net SCL8: now also R27.1, U9.6; no longer R26.1, U9.1
- net SCL9: now also R30.1, U10.6; no longer R29.1, U10.1
- net SDA: now also R1.1, U1.1; no longer R2.1, U1.6
- net SDA1: now also R5.1, U2.1; no longer R6.1, U2.6
- net SDA10: now also R32.1, U11.1; no longer R33.1, U11.6
- net SDA11: now also R35.1, U12.1; no longer R36.1, U12.6
- net SDA12: now also R38.1, U13.1; no longer R39.1, U13.6
- net SDA13: now also R41.1, U14.1; no longer R42.1, U14.6
- net SDA14: now also R44.1, U15.1; no longer R45.1, U15.6
- net SDA15: now also R47.1, U16.1; no longer R48.1, U16.6
- net SDA16: now also R50.1, U17.1; no longer R51.1, U17.6
- net SDA17: now also R53.1, U18.1; no longer R54.1, U18.6
- net SDA18: now also R56.1, U19.1; no longer R57.1, U19.6
- net SDA19: now also R59.1, U20.1; no longer R60.1, U20.6
- net SDA2: now also R8.1, U3.1; no longer R9.1, U3.6
- net SDA20: now also R62.1, U21.1; no longer R63.1, U21.6
- net SDA21: now also R65.1, U22.1; no longer R66.1, U22.6
- net SDA22: now also R68.1, U23.1; no longer R69.1, U23.6
- net SDA23: now also R71.1, U24.1; no longer R72.1, U24.6
- net SDA3: now also R11.1, U4.1; no longer R12.1, U4.6
- net SDA4: now also R14.1, U5.1; no longer R15.1, U5.6
- net SDA5: now also R17.1, U6.1; no longer R18.1, U6.6
- net SDA6: now also R20.1, U7.1; no longer R21.1, U7.6
- net SDA7: now also R23.1, U8.1; no longer R24.1, U8.6
- net SDA8: now also R26.1, U9.1; no longer R27.1, U9.6
- net SDA9: now also R29.1, U10.1; no longer R30.1, U10.6
Routing:
- net SDA3: track 19.1 -> 20.0 mm
- net SDA9: track 19.1 -> 20.0 mm
- net SDA8: track 19.1 -> 20.0 mm
- net SDA7: track 19.1 -> 20.0 mm
- net SDA6: track 19.1 -> 20.0 mm
- net SDA5: track 19.1 -> 20.0 mm
- net SDA4: track 19.1 -> 20.0 mm
- net SDA2: track 19.1 -> 20.0 mm
- net SDA10: track 19.1 -> 20.0 mm
- net SDA1: track 19.1 -> 20.0 mm
- net SDA11: track 19.1 -> 20.0 mm
- net SDA: track 19.1 -> 20.0 mm
- net SDA22: track 19.1 -> 20.0 mm
- net SDA21: track 19.1 -> 20.0 mm
- net SDA19: track 19.1 -> 20.0 mm
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Other:
- board text added: "x02"
- board text removed: "x01"
